File: kicad_jackpad/breakout_jackpad/breakout_jackpad.kicad_pcb (KiCad board)
At the start: 2 copper layers, 42.5 x 41.9 mm, 18 parts, among them J1 ws2812 connect, J10 MR30, J11 jumper cap for 12b, J2 EXTRA, J3 Ext 5v supply, J4 MAX98357A, J8 Conn_01x04_Pin, J9 Conn_01x03_Pin, U1 XIAO_ESP32_S3, U2 74AHCT125

Commit message: Added CAD files for pcb enclosure
Parts:
- added ?: , , F.Cu at (203.5, 120.6)
Changed lines of the file:
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@@
 		)
+	)
+	(footprint ""
+		(layer "F.Cu")
+		(at 203.549271 120.632377)
+		(property "Reference" ""
+			(at 0 0 0)
+			(layer "F.SilkS")
+			(effects
+				(font
+					(size 1.27 1.27)
+				)
+			)
+		)
+		(property "Value" ""
+			(at 0 0 0)
+			(layer "F.Fab")
+			(effects
+				(font
+					(size 1.27 1.27)
+				)
+			)
+		)
+		(property "Datasheet" ""
+			(at 0 0 0)
+			(layer "F.Fab")
+			(hide yes)
+			(effects
+				(font
+					(size 1.27 1.27)
+				)
+			)
+		)
+		(property "Description" ""
+			(at 0 0 0)
+			(layer "F.Fab")
+			(hide yes)
+			(effects
+				(font
+					(size 1.27 1.27)
+				)
+			)
+		)
+		(duplicate_pad_numbers_are_jumpers no)
+		(pad "" np_thru_hole circle
+			(at 0 0)
+			(size 3.2 3.2)
+			(drill 3.2)
+			(layers "*.Cu" "*.Mask")
+		)
+		(embedded_fonts no)
 	)
 	(footprint "Connector_PinSocket_2.54mm:PinSocket_1x04_P2.54mm_Vertical"
