File: kicad_jackpad/breakout_jackpad/slot_jackpad/slot_jackpad.kicad_pcb (KiCad board)
At the start: 2 copper layers, 41.6 x 45 mm, 18 parts, among them J1 DRV8833, J2 i2c, J3 meow, J4 MR30 OUT, J5 MR30 IN, J6 Conn_01x04_Pin, J7 Conn_01x03_Pin, SW1 white_v2, U1 ESP32-C3_SUPERMINI_TH

Commit message: Added CAD files for pcb enclosure
Parts:
- added REF**: MountingHole_2.2mm_M2, MountingHole:MountingHole_2.2mm_M2, F.Cu at (156.4, 83.3)
- added REF**: MountingHole_2.2mm_M2, MountingHole:MountingHole_2.2mm_M2, F.Cu at (123.3, 124.7)
- added REF**: MountingHole_2.2mm_M2, MountingHole:MountingHole_2.2mm_M2, F.Cu at (118.3, 82.9)
- added REF**: MountingHole_2.2mm_M2, MountingHole:MountingHole_2.2mm_M2, F.Cu at (152.1, 124.8)
